Commit message: Add files via upload

File: track_v1/urdf/track_v1.urdf (robot description, URDF)
Before this commit: robot track_v1, 2 links, 1 joints
Links:
- link base_link: geometry collision mesh filename=package://track_v1/meshes/base_link.STL; visual mesh filename=package://track_v1/meshes/base_link.STL
- link track_link: geometry collision mesh filename=package://track_v1/meshes/track_link.STL; visual mesh filename=package://track_v1/meshes/track_link.STL
Joints:
- joint track_joint: type fixed -> prismatic
