Commit message: update track3

File: track3_v1/urdf/track3_v1.urdf (robot description, URDF)
Before this commit: robot track3_v1, 15 links, 14 joints
Links:
- link track_Link: geometry collision mesh filename=package://track3_v1/meshes/track3_v1.dae; visual mesh filename=package://track3_v1/meshes/track3_v1.dae
Joints:
- joint gree_joint: axis 0 0 0 -> 0 0 -1; limit (none) -> lower=0 upper=0 effort=0 velocity=0; type fixed -> prismatic
